File: pcb/boost.brick.kicad_pcb (KiCad board)
At the start: 2 copper layers, 0 parts

Commit message: Add first prototype
Parts:
- added BT1: Battery_Cell, Battery:BatteryHolder_Keystone_2460_1xAA, B.Cu at (130.0, 106.0)
- added C1: 10u, Capacitor_SMD:C_0805_2012Metric, F.Cu at (135.0, 108.0)
- added C2: 10u, Capacitor_SMD:C_0805_2012Metric, F.Cu at (139.0, 102.0)
- added L1: 4.7u, Inductor_SMD:L_Taiyo-Yuden_NR-30xx, F.Cu at (135.0, 104.5)
- added R1: 120k, Resistor_SMD:R_0805_2012Metric, F.Cu at (143.0, 102.0)
- added R2: 15k, Resistor_SMD:R_0805_2012Metric, F.Cu at (143.0, 105.0)
- added R3: 120k, Resistor_SMD:R_0805_2012Metric, F.Cu at (143.0, 108.0)
- added TP1: VBat, TestPoint:TestPoint_THTPad_D2.0mm_Drill1.0mm, F.Cu at (125.0, 104.0)
- added TP2: EN, TestPoint:TestPoint_THTPad_D2.0mm_Drill1.0mm, F.Cu at (125.0, 108.0)
- added TP3: VOut, TestPoint:TestPoint_THTPad_D3.0mm_Drill1.5mm, F.Cu at (121.0, 100.0)
- added TP4: GND, TestPoint:TestPoint_THTPad_D3.0mm_Drill1.5mm, F.Cu at (121.0, 112.0)
- added U1: TPS61220DCK, Package_TO_SOT_SMD:Texas_R-PDSO-G6, F.Cu at (139.0, 105.0)
- added kibuzzard-64C6B850: G***, kibuzzard-64C6B850, F.Cu at (128.0, 100.0)
- added kibuzzard-64C6B99F: G***, kibuzzard-64C6B99F, F.Cu at (127.0, 112.0)
- added kibuzzard-64C6BA9D: G***, kibuzzard-64C6BA9D, F.Cu at (129.7, 102.9)
- added kibuzzard-64C6BAA4: G***, kibuzzard-64C6BAA4, F.Cu at (129.7, 109.0)
- added kibuzzard-64ECEE1E: G***, kibuzzard-64ECEE1E, B.Cu at (123.0, 100.0)
- added kibuzzard-64ECEE9B: G***, kibuzzard-64ECEE9B, B.Cu at (123.0, 112.0)
Routing:
- net Net-(U1-VOUT): track 0.00 -> 29.8 mm, vias 0 -> 2
- net Net-(BT1-+): track 0.00 -> 24.5 mm, vias 0 -> 1
- net Net-(U1-EN): track 0.00 -> 15.2 mm, vias 0 -> 1
- net Net-(U1-FB): track 0.00 -> 7.99 mm
- net Net-(U1-L): track 0.00 -> 1.80 mm
- net GND: vias 0 -> 11
- added copper zone on B.Cu, net GND
- added copper zone on F.Cu, net GND
Other:
- board outline added: 67 x 18 mm
- board text added: "Bottom Assembly View | Scale 1:1"
- board text added: "Top Assembly View | Scale 1:1"
- board text added: "boost.brick.AA"
- board text added: "v1.0.0 (c) by cazaugg"
