File: pcb/boost.brick.kicad_sch (KiCad schematic)
At the start: 1 part

Commit message: Add first prototype
Parts:
- added BT1: Battery_Cell, Battery:BatteryHolder_Keystone_2460_1xAA, symbol Device:Battery_Cell
- added C1, C2: 10u, Capacitor_SMD:C_0805_2012Metric, symbol Device:C
- added L1: 4.7u, Inductor_SMD:L_Taiyo-Yuden_NR-30xx, symbol Device:L_Iron
- added R2: 15k, Resistor_SMD:R_0805_2012Metric, symbol Device:R
- added R3: 120k, Resistor_SMD:R_0805_2012Metric, symbol Device:R
- added TP1: VBat, TestPoint:TestPoint_THTPad_D2.0mm_Drill1.0mm, symbol Connector:TestPoint
- added TP2: EN, TestPoint:TestPoint_THTPad_D2.0mm_Drill1.0mm, symbol Connector:TestPoint
- added TP3: VOut, TestPoint:TestPoint_THTPad_D3.0mm_Drill1.5mm, symbol Connector:TestPoint
- added TP4: GND, TestPoint:TestPoint_THTPad_D3.0mm_Drill1.5mm, symbol Connector:TestPoint
- added U1: TPS61220DCK, Package_TO_SOT_SMD:Texas_R-PDSO-G6, symbol Regulator_Switching:TPS61220DCK
- R1: renamed from R?; value R -> 120k; footprint (none) -> Resistor_SMD:R_0805_2012Metric; Specs (none) -> 1%, 1/8W
Connections:
- net at R1.1: now also R2.2, R3.2, U1.2 (FB)
- net at R1.2: now also C2.1, TP3.1, U1.4 (VOUT)
- new net: TP2.1, U1.6 (EN)
- new net: BT1.1 (+), C1.1, L1.1, TP1.1, U1.1 (VIN)
- new net: L1.2, U1.5 (L)
- new net GND: BT1.2 (-), C1.2, C2.2, R2.1, R3.1, TP4.1, U1.3 (GND)
Other:
- note added: "| VOUT | R1 | R2 | R3 | ------------------------------ | +5V | 120k | 15k | 120k | | +3.3V | 56k | 10k | None | | +3.0V | 100k | 22k | 220k | | +2.5V | 120k | 33k | 330k | | +2.0V | 150k | 100k | 100k | | +1.8V | 39k | 15k | None |"
- moved on the sheet: R1
